File: kicad/dram-tester.kicad_pcb (KiCad board)
At the start: 2 copper layers, 56.5 x 43.2 mm, 8 parts, among them U1 TMM41256AP

Commit message: minor fixes
Parts:
- moved C1 2.82 mm to (170.8, 76.2), turned to 0 degrees
- moved D2 1.24 mm to (172.2, 92.7)
- moved R1 1.24 mm to (172.2, 102.8)
- moved D1 1.24 mm to (172.2, 100.3)
- moved R2 1.24 mm to (172.2, 90.1)
Connections:
- A2 pad 19: /CAS -> /RAS
- A2 pad 20: /RAS -> /CAS
- A2 pad 27: unconnected-(A2-+5V-Pad27) -> VCC
Routing:
- net VCC: track 0.00 -> 79.9 mm
- net /CAS: track 0.00 -> 37.4 mm
- net /A8: track 20.1 -> 0.00 mm
- net Net-(A2-A3): track 49.9 -> 55.6 mm
- net Net-(A2-A2): track 49.9 -> 55.0 mm
- net Net-(A2-A4): track 31.2 -> 35.2 mm
- net /RAS: track 42.7 -> 44.8 mm
- net /A0: track 22.2 -> 21.2 mm
- net /A2: track 21.2 -> 20.1 mm
- net /DOUT: track 29.7 -> 30.3 mm
- added copper zone on F.Cu, net GND
- removed copper zone on F.Cu, net VCC

Commit message: add logos
Parts:
- added G***: LOGO, dram_tester:cc-by-sa-logo, B.Cu at (150.6, 102.1)
- added REF**: OSHW-Logo_11.4x12mm_SilkScreen, Symbol:OSHW-Logo_11.4x12mm_SilkScreen, B.Cu at (162.6, 107.4)

Commit message: fix A8 trace
Routing:
- net /A8: track 0.00 -> 20.1 mm
Changed lines of the file:
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@@
 			(net 18 "unconnected-(A2-D1{slash}TX-Pad1)")
 			(pinfunction "D1/TX")
-			(pintype "bidirectional")
+			(pintype "bidirectional+no_connect")
 		)
 		(pad "2" thru_hole oval
@@
 			(net 15 "unconnected-(A2-D0{slash}RX-Pad2)")
 			(pinfunction "D0/RX")
-			(pintype "bidirectional")
+			(pintype "bidirectional+no_connect")
 		)
 		(pad "3" thru_hole oval
@@
 			(net 16 "unconnected-(A2-~{RESET}-Pad3)")
 			(pinfunction "~{RESET}")
-			(pintype "input")
+			(pintype "input+no_connect")
 		)
 		(pad "4" thru_hole oval
@@
 			(net 9 "unconnected-(A2-3V3-Pad17)")
 			(pinfunction "3V3")
-			(pintype "power_out")
+			(pintype "power_out+no_connect")
 		)
 		(pad "18" thru_hole oval
@@
 			(net 5 "unconnected-(A2-AREF-Pad18)")
 			(pinfunction "AREF")
-			(pintype "input")
+			(pintype "input+no_connect")
 		)
 		(pad "19" thru_hole oval
@@
 			(net 31 "unconnected-(A2-A5-Pad24)")
 			(pinfunction "A5")
-			(pintype "bidirectional")
+			(pintype "bidirectional+no_connect")
 		)
 		(pad "25" thru_hole oval
@@
 			(net 8 "unconnected-(A2-A6-Pad25)")
 			(pinfunction "A6")
-			(pintype "bidirectional")
+			(pintype "bidirectional+no_connect")
 		)
 		(pad "26" thru_hole oval
@@
 			(net 22 "unconnected-(A2-A7-Pad26)")
 			(pinfunction "A7")
-			(pintype "bidirectional")
+			(pintype "bidirectional+no_connect")
 		)
 		(pad "27" thru_hole oval
@@
 			(net 23 "unconnected-(A2-~{RESET}-Pad28)")
 			(pinfunction "~{RESET}")
-			(pintype "input")
+			(pintype "input+no_connect")
 		)
 		(pad "29" thru_hole oval
@@
 			(net 13 "unconnected-(A2-VIN-Pad30)")
 			(pinfunction "VIN")
-			(pintype "power_in")
+			(pintype "power_in+no_connect")
 		)
 		(embedded_fonts no)
@@
 	)
 	(segment
+		(start 161.29 101.6)
+		(end 163.83 99.06)
+		(width 0.2)
+		(layer "F.Cu")
+		(net 26)
+	)
+	(segment
+		(start 144.78 101.6)
+		(end 161.29 101.6)
+		(width 0.2)
+		(layer "F.Cu")
+		(net 26)
+	)
+	(segment
