File: kicad/dram-tester.kicad_sch (KiCad schematic)
At the start: 8 parts, among them U1 TMM41256AP

Commit message: minor fixes
Connections:
- net CAS: now also A2.20 (A1); no longer A2.19 (A0)
- net RAS: now also A2.19 (A0); no longer A2.20 (A1)
- net VCC: now also A2.27 (+5V)
Changed lines of the file:
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@@
 	)
 	(label "CAS"
-		(at 144.78 128.27 0)
+		(at 144.78 130.81 0)
 		(effects
 			(font
@@
 	)
 	(label "RAS"
-		(at 144.78 130.81 0)
+		(at 144.78 128.27 0)
 		(effects
 			(font
@@
 	(symbol
 		(lib_id "power:VCC")
-		(at 135.89 105.41 0)
+		(at 135.89 102.87 0)
 		(unit 1)
 		(exclude_from_sim no)
@@
 		(fields_autoplaced yes)
 		(property "Reference" "#PWR06"
-			(at 135.89 109.22 0)
+			(at 135.89 106.68 0)
 			(effects
 				(font
@@
 		)
 		(property "Value" "VCC"
-			(at 135.89 101.2769 0)
+			(at 135.89 98.7369 0)
 			(effects
 				(font
@@
 		)
 		(property "Footprint" ""
-			(at 135.89 105.41 0)
+			(at 135.89 102.87 0)
 			(effects
 				(font
@@
 		)
 		(property "Datasheet" ""
-			(at 135.89 105.41 0)
+			(at 135.89 102.87 0)
 			(effects
 				(font
@@
 		)
 		(property "Description" "Power symbol creates a global label with name \"VCC\""
-			(at 135.89 105.41 0)
-			(effects
-				(font
+			(at 135.89 102.87 0)
+			(effects
+				(font

Commit message: fix A8 trace
Connections:
- no-connect marks 0 -> 10
Changed lines of the file:
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@@
 		(color 0 0 0 0)
+	)
+	(no_connect
+		(at 143.51 113.03)
+	)
+	(no_connect
+		(at 118.11 113.03)
+	)
+	(no_connect
+		(at 143.51 146.05)
+	)
+	(no_connect
+		(at 143.51 143.51)
+	)
+	(no_connect
+		(at 128.27 102.87)
+	)
+	(no_connect
+		(at 118.11 115.57)
+	)
+	(no_connect
+		(at 133.35 102.87)
+	)
+	(no_connect
+		(at 143.51 115.57)
+	)
+	(no_connect
+		(at 143.51 140.97)
+	)
+	(no_connect
+		(at 143.51 123.19)
 	)
 	(bus_entry
